File: PCB/MonpolyElectronicV2/MonpolyElectronicV2.kicad_pcb (KiCad board)
At the start: 2 copper layers, 93.3 x 128.4 mm, 102 parts, among them J1 Conn_01x14, J10 Conn_01x01, J12 Conn_01x01, J13 Conn_01x01, J14 Conn_01x01, J15 Conn_01x01, J16 Conn_01x01, J18 Conn_01x01, J19 Conn_01x01, J2 10155435-00011LF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

Commit message: base done
Parts:
- added J6: Conn_01x02, Connector_JST:JST_XH_B2B-XH-A_1x02_P2.50mm_Vertical, F.Cu at (109.0, 40.0)
- added J9: Conn_01x02, Connector_PinHeader_2.54mm:PinHeader_1x02_P2.54mm_Vertical, F.Cu at (109.0, 35.0)
Routing:
- net BAT: track 38.8 -> 51.9 mm
- net GND: track 121.9 -> 126.9 mm
